File: Circuitry/KiCad/Cube Solver/Motor Breakout/Motor Breakout.kicad_pcb (KiCad board)
At the start: 2 copper layers, 36 x 52 mm, 13 parts, among them J2 Motor Input, J3 Motherboard Breakout, J4 Servo Input, J5 Servo Output, J6 Encoder Input

Commit message: Motors confirmed working
Other:
- board text added: "3.3V GND SDA SCL"
- board text removed: "3.3V GND SCL SDA"
Changed lines of the file:
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@@
 		)
 	)
-	(gr_text "3.3V GND SCL SDA"
+	(gr_text "3.3V GND SDA SCL"
 		(at 113.6 38.8 0)
 		(layer "F.SilkS")
